Commit message: * WIP : latest updates

File: src/futurakart/futurakart_description/urdf/futurakart.urdf (robot description, URDF)
Before this commit: robot futurakart, 2 links, 1 joints
Links:
- removed link chassis_link
- added link base_footprint
- link base_link: geometry visual box size=${base_length} ${base_width} ${base_height}
Joints:
- joint base_link_joint: child chassis_link -> base_link; origin xyz=0 0 0 rpy=0 0 0 -> xyz=0 0 ${vertical_offset}; parent base_link -> base_footprint

Commit message: * modify urdf file : dimension and position of the model

File: src/futurakart/futurakart_description/urdf/futurakart.urdf (robot description, URDF)
Before this commit: robot futurakart, 2 links, 1 joints
Links:
- link base_link: geometry visual box size=${base_width} ${base_length} ${base_height}
Joints:
- joint base_link_joint: origin xyz=0 0 ${vertical_offset} -> xyz=0 ${track/2} -${vertical_offset}

Commit message: * Update README
* Update 'control' conf

* Modify urdf

File: src/futurakart/futurakart_description/urdf/futurakart.urdf (robot description, URDF)
Before this commit: robot futurakart, 2 links, 1 joints
Joints:
- joint base_link_joint: origin xyz=0 ${track/2} -${vertical_offset} -> xyz=0 -${track/2} ${vertical_offset}

Commit message: * Update futurakart messages, remove previous ones
* Adapt simulator and futurakart_base node to new messages

* Activate EKF robot localization

File: src/futurakart/futurakart_description/urdf/futurakart.urdf (robot description, URDF)
Before this commit: robot futurakart, 2 links, 1 joints
Joints:
- joint base_link_joint: child base_link -> base_footprint; origin xyz=0 -${track/2} ${vertical_offset} -> xyz=0 ${track/2} -${vertical_offset}; parent base_footprint -> base_link

Commit message: * Add complete base.launch emulation in mbed emulator
* Add verbose argument in emulator

* [DEV] Fix description axis problems

File: src/futurakart/futurakart_description/urdf/futurakart.urdf (robot description, URDF)
Before this commit: robot futurakart, 2 links, 1 joints
Links:
- link base_link: geometry visual box size=${base_length} ${base_width} ${base_height}
Joints:
- joint base_link_joint: origin xyz=0 ${track/2} -${vertical_offset} -> xyz=${track/2} 0 -${vertical_offset}

Commit message: * Change base_link to front wheel base
* Copy teleop config to local

File: src/futurakart/futurakart_description/urdf/futurakart.urdf (robot description, URDF)
Before this commit: robot futurakart, 2 links, 1 joints
Joints:
- joint base_link_joint: origin xyz=${track/2} 0 -${vertical_offset} -> xyz=-${track/2} 0 -${vertical_offset}

Commit message: * Remove absolute path from map file
* Fix robot localization params

* Fix urdf for Gazebo simulation

* [WIP] Stage simulation

File: src/futurakart/futurakart_description/urdf/futurakart.urdf (robot description, URDF)
Before this commit: robot futurakart, 2 links, 1 joints
Links:
- added link chassis_link, mass 16.523; visual box size=${base_length} ${base_width} ${base_height}
- link base_link: geometry 
Joints:
- removed joint base_link_joint
- added joint base_footprint_link_joint: type fixed, parent base_link, child base_footprint, origin xyz=-${track/2} 0 -${vertical_offset}
- added joint chassis_link_joint: type fixed, parent base_link, child chassis_link, origin xyz=-${track/2} 0 ${wheel_radius}

Commit message: * Rename wheelbase <-> track
* [WIP] Update params in teb_local_planner

File: src/futurakart/futurakart_description/urdf/futurakart.urdf (robot description, URDF)
Before this commit: robot futurakart, 3 links, 2 joints
Joints:
- joint base_footprint_link_joint: origin xyz=-${track/2} 0 -${vertical_offset} -> xyz=-${wheelbase/2} 0 -${vertical_offset}
- joint chassis_link_joint: origin xyz=-${track/2} 0 ${wheel_radius} -> xyz=-${wheelbase/2} 0 ${wheel_radius}

Commit message: *[WIP] Update urdf => Problems with Gazebo and Mbed emulation !

File: src/futurakart/futurakart_description/urdf/futurakart.urdf (robot description, URDF)
Before this commit: robot futurakart, 3 links, 2 joints
Links:
- added link rear_track_link, mass 0.3; visual cylinder length=${track_rear} radius=0.005
- link chassis_link: mass 16.523 -> 5.0
Joints:
- added joint rear_track_joint: type fixed, parent base_link, child rear_track_link, origin xyz=-${wheelbase} 0 0

Commit message: *[WIP] Update robot HW to accept steering arm *[WIP] Update urdf model => front wheels are not controlled

File: src/futurakart/futurakart_description/urdf/futurakart.urdf (robot description, URDF)
Before this commit: robot futurakart, 4 links, 3 joints
Joints:
- joint chassis_link_joint: origin xyz=-${wheelbase/2} 0 ${wheel_radius} -> xyz=-${wheelbase/2} 0 ${wheel_radius + base_height}
